Commit message: Working Lidar

File: description/imu.xacro (robot description, xacro)
@@ -16,5 +16,5 @@
     <parent link="base_link"/>
     <child link="imu_link"/>
-    <origin xyz="0.28 -0.260 0.49071"/>
+    <origin xyz="0.28 -0.260 0.150" rpy="0 0 3.14159"/>
   </joint>
   <gazebo reference="imu_link">

File: description/lidar.xacro (robot description, xacro)
@@ -4,5 +4,5 @@
         <parent link="base_link"/>
         <child link="laser_frame"/>
-        <origin xyz="0.28 0.255 0.57071" rpy="0 0 0"/>
+        <origin xyz="0.28 0.255 0.225" rpy="0 0 0"/>
     </joint>
     <link name="laser_frame">

File: description/robot_core.xacro (robot description, xacro)
@@ -18,21 +18,20 @@
     </material>
     <!-- BASE LINK -->
-    <link name="base_link">
-    </link>
+    <!-- <link name="base_link" /> -->
+    <joint name="base_footprint_joint" type="fixed">
+        <parent link="base_footprint"/>
+        <child link="base_link"/>
+        <origin xyz="0 0 0.35571" rpy="0 0 3.14159"/>
+    </joint>
     <!-- BASE_FOOTPRINT LINK -->
-    <joint name="base_footprint_joint" type="fixed">
-        <parent link="base_link"/>
-        <child link="base_footprint"/>
-        <origin xyz="0 0 0" rpy="0 0 0"/>
-    </joint>
     <link name="base_footprint">
     </link>
     <!-- Chassis Link -->
-    <joint name="chassis_joint" type="fixed">
+    <!-- <joint name="chassis_joint" type="fixed">
         <parent link="base_link"/>
         <child link="chassis"/>
-        <origin xyz="0 0 0.34571"/>
-    </joint>
-    <link name="chassis">
+        <origin xyz="0 0 0"/>
+    </joint> -->
+    <link name="base_link">
         <visual>
             <origin xyz ="0 0 0"/>
@@ -59,5 +58,5 @@
         <parent link="base_link" />
         <child link="front_left_wheel" />
-        <origin xyz ="0.44071 -0.44259 0.15" rpy="-${pi/2} 0 0" />
+        <origin xyz ="0.42 0.47 -0.19821" rpy="-${pi/2} 0 0" />
         <axis xyz="0 0 1" />
     </joint>
@@ -65,5 +64,5 @@
         <visual>
             <geometry>
-                <cylinder radius="0.15" length="0.09" />
+                <cylinder radius="0.1575" length="0.09" />
             </geometry>
             <material name="blue"/>
@@ -71,8 +70,8 @@
         <collision>
             <geometry>
-                <cylinder radius="0.15" length="0.09" />
+                <cylinder radius="0.1575" length="0.09" />
             </geometry>
         </collision>
-        <xacro:inertial_cylinder mass="1.2" length="0.09" radius="0.15">
+        <xacro:inertial_cylinder mass="1.2" length="0.09" radius="0.1575">
             <origin xyz="0 0 0" rpy="0 0 0"/>
         </xacro:inertial_cylinder>
@@ -87,5 +86,5 @@
         <parent link="base_link" />
         <child link="front_right_wheel" />
-        <origin xyz ="0.44071 0.44259 0.15" rpy="${pi/2} 0 0" />
+        <origin xyz ="0.42 -0.47 -0.19821" rpy="${pi/2} 0 0" />
         <axis xyz="0 0 -1" />
     </joint>
@@ -93,5 +92,5 @@
         <visual>
             <geometry>
-                <cylinder radius="0.15" length="0.09" />
+                <cylinder radius="0.1575" length="0.09" />
             </geometry>
             <material name="blue"/>
@@ -99,8 +98,8 @@
         <collision>
             <geometry>
-                <cylinder radius="0.15" length="0.09" />
+                <cylinder radius="0.1575" length="0.09" />
             </geometry>
         </collision>
-        <xacro:inertial_cylinder mass="1.2" length="0.09" radius="0.15">
+        <xacro:inertial_cylinder mass="1.2" length="0.09" radius="0.1575">
             <origin xyz="0 0 0" rpy="0 0 0"/>
         </xacro:inertial_cylinder>
@@ -115,5 +114,5 @@
         <parent link="base_link" />
         <child link="back_left_wheel" />
-        <origin xyz ="-0.44071 -0.44259 0.15" rpy="-${pi/2} 0 0" />
+        <origin xyz ="-0.42 0.47 -0.19821" rpy="-${pi/2} 0 0" />
         <axis xyz="0 0 1" />
     </joint>
@@ -121,5 +120,5 @@
         <visual>
             <geometry>
-                <cylinder radius="0.15" length="0.09" />
+                <cylinder radius="0.1575" length="0.09" />
             </geometry>
             <material name="blue"/>
@@ -127,8 +126,8 @@
         <collision>
             <geometry>
-                <cylinder radius="0.15" length="0.09" />
+                <cylinder radius="0.1575" length="0.09" />
             </geometry>
         </collision>
-        <xacro:inertial_cylinder mass="1.2" length="0.09" radius="0.15">
+        <xacro:inertial_cylinder mass="1.2" length="0.09" radius="0.1575">
             <origin xyz="0 0 0" rpy="0 0 0"/>
         </xacro:inertial_cylinder>
@@ -143,5 +142,5 @@
         <parent link="base_link" />
         <child link="back_right_wheel" />
-        <origin xyz ="-0.44071 0.44259 0.15" rpy="${pi/2} 0 0" />
+        <origin xyz ="-0.42 -0.47 -0.19821" rpy="${pi/2} 0 0" />
         <axis xyz="0 0 -1" />
     </joint>
@@ -149,5 +148,5 @@
         <visual>
             <geometry>
-                <cylinder radius="0.15" length="0.09" />
+                <cylinder radius="0.1575" length="0.09" />
             </geometry>
             <material name="blue"/>
@@ -155,8 +154,8 @@
         <collision>
             <geometry>
-                <cylinder radius="0.15" length="0.09" />
+                <cylinder radius="0.1575" length="0.09" />
             </geometry>
         </collision>
-        <xacro:inertial_cylinder mass="1.2" length="0.09" radius="0.15">
+        <xacro:inertial_cylinder mass="1.2" length="0.09" radius="0.1575">
             <origin xyz="0 0 0" rpy="0 0 0"/>
         </xacro:inertial_cylinder>
